File: pcb/analog_bms/analog_bms.kicad_sch (KiCad schematic)
At the start: 51 parts, among them J1 Screw_Terminal_1x2, J2 MODULE+, J3 MODULE-, Q1 PMOS, Q2 NMOS, Q3 PMOS, Q4 NMOS, Q5 PMOS, U1 TLV7031DBV, U2 TLV7031DBV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

Commit message: Digikey, TI, and PCBWay orders!
Parts:
- R1: value Thermistor_PTC -> Thermistor_NTC
Changed lines of the file:
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@@
 			)
 		)
-		(property "Value" "Thermistor_PTC"
+		(property "Value" "Thermistor_NTC"
 			(at 57.4675 162.56 90)
 			(effects

Commit message: LTspice sim + attempt at fixing OV UV dividers
Parts:
- R11: value 100 -> 100k
Changed lines of the file:
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@@
 			)
 		)
-		(property "Value" "100"
+		(property "Value" "100k"
 			(at 77.978 134.62 90)
 			(effects

Commit message: Fixed OV divider & Q3/5 pulldown stronger
Parts:
- R12: value R -> 1M; now fitted
Changed lines of the file:
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@@
 		(in_bom yes)
 		(on_board yes)
-		(dnp yes)
+		(dnp no)
 		(property "Reference" "R12"
 			(at 86.868 124.46 90)
@@
 			)
 		)
-		(property "Value" "R"
+		(property "Value" "1M"
 			(at 86.868 127 90)
 			(effects
